File: air_foil_pcb/air_foil_pcb.kicad_pcb (KiCad board)
At the start: 4 copper layers, 76.2 x 170.2 mm, 244 parts, among them J2 Tube Connector, J3 Brass Manifold, J4 End_plate_mount, J5 Conn_01x10, U1 TCA9548APWR, U10 HSCDRRN400MD2A3, U11 HSCDRRN400MD2A3, U12 HSCDRRN400MD2A3, U13 HSCDRRN400MD2A3, U14 TCA9548APWR, U15 HSCDRRN400MD2A3, U16 HSCDRRN400MD2A3, U17 HSCDRRN400MD2A3, U18 HSCDRRN400MD2A3, U19 HSCDRRN400MD2A3, U2 HSCDRRN400MD2A3, U20 HSCDRRN400MD2A3, U21 HSCDRRN400MD2A3, U22 HSCDRRN400MD2A3, U23 TCA9548APWR, U24 HSCDRRN400MD2A3, U25 HSCDRRN400MD2A3, U26 HSCDRRN400MD2A3, U27 HSCDRRN400MD2A3, U28 HSCDRRN400MD2A3, U29 HSCDRRN400MD2A3, U3 HSCDRRN400MD2A3, U30 HSCDRRN400MD2A3, U31 HSCDRRN400MD2A3, U32 TCA9548APWR, U33 HSCDRRN400MD2A3, U34 HSCDRRN400MD2A3, U35 HSCDRRN400MD2A3, U36 HSCDRRN400MD2A3, U4 HSCDRRN400MD2A3, U5 HSCDRRN400MD2A3, U6 HSCDRRN400MD2A3, U7 HSCDRRN400MD2A3, U8 HSCDRRN400MD2A3, U9 HSCDRRN400MD2A3

Commit message: finished layout
Parts:
- JP31, JP32, JP33, JP34, JP35, JP36, JP37, JP38, JP47, JP48, JP49, JP50, JP51, JP52, JP53, JP54, JP63, JP64, JP65, JP66, JP67, JP68, JP69, JP70, U28: moved to B.Cu
- U34: moved to F.Cu
- moved JP40 135.4 mm to (77.9, 71.2)
- moved JP50 130.7 mm to (81.3, 62.1), turned to 180 degrees
- moved C16 128.7 mm to (84.9, 122.1), turned to -90 degrees
- moved JP44 127.8 mm to (81.4, 71.2)
- moved C20 124.3 mm to (76.7, 133.8), turned to -90 degrees
- moved JP41 121.9 mm to (60.8, 71.4)
- moved C48 120.3 mm to (85.7, 122.2), turned to -90 degrees
- moved JP54 119.0 mm to (81.3, 59.3), turned to 180 degrees
- moved JP60 117.8 mm to (77.1, 48.9)
- moved C15 115.2 mm to (67.6, 122.2), turned to -90 degrees
- moved C52 115.2 mm to (75.9, 133.8), turned to -90 degrees
- moved JP51 114.1 mm to (63.8, 59.0), turned to 180 degrees
- moved R24 113.4 mm to (82.7, 132.4), turned to 90 degrees
- moved JP45 113.3 mm to (64.3, 71.4)
- moved C72 112.1 mm to (95.7, 52.1), turned to -90 degrees
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Routing:
- net +3V3: track 77.2 -> 239.2 mm, vias 24 -> 74
- net GND: track 64.2 -> 202.0 mm, vias 14 -> 17
- net /C37: track 0.00 -> 82.3 mm, vias 0 -> 2
- net /D37: track 0.00 -> 80.8 mm, vias 0 -> 2
- net /D33: track 0.00 -> 78.8 mm, vias 0 -> 3
- net /C32: track 0.00 -> 76.1 mm, vias 0 -> 1
- net /C24: track 0.00 -> 75.2 mm, vias 0 -> 2
- net /C33: track 0.00 -> 74.0 mm, vias 0 -> 2
- net /D32: track 0.00 -> 69.3 mm, vias 0 -> 1
- net /D24: track 0.00 -> 69.3 mm, vias 0 -> 2
- net /C36: track 0.00 -> 62.7 mm, vias 0 -> 2
- net /D36: track 0.00 -> 62.0 mm, vias 0 -> 2
- net /C31: track 0.00 -> 61.7 mm, vias 0 -> 2
- net /D13: track 0.00 -> 57.3 mm, vias 0 -> 3
- net /C13: track 0.00 -> 57.2 mm, vias 0 -> 2
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Other:
- board text added: "3V3"
- board text added: "GND"
- board text added: "M0 0x70"
- board text added: "M1 0x71"
- board text added: "M2 0x72"
- board text added: "M3 0x74"
- board text added: "RES_0"
- board text added: "RES_1"
- board text added: "RES_2"
- board text added: "RES_3"
- board text added: "S00"
- board text added: "S01"
- board text added: "S02"
- board text added: "S03"
- board text added: "S04"
- board text added: "S05"
- board text added: "S06"
- board text added: "S07"
- board text added: "S10"
- board text added: "S11"
- board text added: "S12"
- board text added: "S13"
- board text added: "S14"
- board text added: "S15"
- board text added: "S16"
- board text added: "S17"
- board text added: "S20"
- board text added: "S21"
- board text added: "S22"
- board text added: "S23"
- board text added: "S24"
- board text added: "S25"
- board text added: "S26"
- board text added: "S27"
- board text added: "S30"
- board text added: "S31"
- board text added: "S32"
- board text added: "S33"
- board text added: "S34"
- board text added: "S35"
- board text added: "S36"
- board text added: "S37"
- board text added: "SCL"
- board text added: "SDA"
